File: hw/FreshTwinkie_v0.1/FreshTwinkie.kicad_pcb (KiCad board)
At the start: 4 copper layers, 45.2 x 17.4 mm, 57 parts, among them J1 USB_B_Micro, J2 USB_C_Receptacle, P1 USB_C_Plug, Q1 PMDXB600UNE, Q2 PMDXB600UNE, Q3 PMDXB600UNE, Q4 Q_NMOS_DGS, U1 INA231, U2 INA231, U3 NCP167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

Commit message: initial remix
Parts:
- removed G***: LOGO, logo
- removed G***: LOGO, gkl_logos:oshw_small
- removed G***: LOGO, gkl_logos:gsd_logo_small
- removed REF** (x4): TestPoint_Pad_D1.0mm, TestPoint:TestPoint_Pad_D1.0mm
- removed U1, U2: INA231, gkl_housings_bga:DSBGA-12_1.56x1.39mm_Layout3x4_P0.4mm
- added U6: INA237, Package_SO:VSSOP-10_3x3mm_P0.5mm, F.Cu at (133.9, 93.3)
- added U7: INA237, Package_SO:VSSOP-10_3x3mm_P0.5mm, F.Cu at (141.7, 93.3)
Connections:
- U5 pad 2: Net-(U5-Pad2) -> unconnected-(U5-PC13-Pad2)
- U5 pad 21: Net-(U5-Pad21) -> unconnected-(U5-PB10-Pad21)
- U5 pad 25: Net-(U5-Pad25) -> unconnected-(U5-PB12-Pad25)
Other:
- board size 45.2 x 17.4 mm -> 45.2 x 23.4 mm
- net class Default removed
