File: hw/FreshTwinkie.kicad_sch (KiCad schematic)
At the start: 50 parts, among them J1 USB_B_Micro, J2 USB_C_Receptacle, P1 USB_C_Plug, Q1 PMDXB600UNE, Q2 PMDXB600UNE, Q3 PMDXB600UNE, Q4 Q_NMOS_DGS, U3 NCP167, U4 AD8606ACB, U5 STM32F072CBUx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

Commit message: wip with rules, 6 layer
Parts:
- added TP1, TP2, TP3, TP4, TP5, TP6, TP7: TestPoint, TestPoint:TestPoint_Pad_D1.0mm, symbol Connector:TestPoint
Connections:
- net CC1_RP1A5: now also U5.2 (PC13); no longer U5.37 (PA14)
- net CC1_RPUSB: now also U5.21 (PB10); no longer U5.34 (PA13)
- net GND: now also TP5.1
- net SCL: now also TP6.1
- net SDA: now also TP7.1
- net UART_RX: now also TP2.1
- net UART_TX: now also TP1.1
- net USB_C_CC2: now also R2.1; no longer R2.4
- net USB_C_CC2_N: now also R2.3; no longer R2.2
- net USB_C_CC2_P: now also R2.4; no longer R2.1
- net USB_C_VBUS_N: now also R1.3; no longer R1.1
- net USB_C_VBUS_P: now also R1.4; no longer R1.2
- net at P1.A4 (VBUS), P1.A9 (VBUS), P1.B4 (VBUS)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: now also R1.2; no longer R1.4
- net at P1.B5 (VCONN): now also R2.2; no longer R2.3
- net at J2.A4 (VBUS), J2.A9 (VBUS), J2.B4 (VBUS)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: now also R1.1; no longer R1.3
- new net SWCLK: TP4.1, U5.37 (PA14)
- new net SWDIO: TP3.1, U5.34 (PA13)
Other:
- note added: "If it is necessary to change layers when routing the USB SuperSpeed signals, place a pair of ground vias close to the transition"
- note added: "Orig:CC1_RP1A5 New:PA14-SWCLK"
- note added: "Orig:CC1_RPUSB New:PA13-SWDIO"
- note added: "Route all USB SuperSpeed signals with 90Ω differential impedance traces without stubs. It is preferred to route these USB SuperSpeed signals on the Top Layer with the Inner Layer 2 being a solid Ground plane as their reference. These signals should not cross a plane split"
- note added: "The CC signals should be routed as single-ended traces with 50Ω impedance. Do not route the CC signals as a differential pair. The CC signals are sensitive so they should be routed without stubs across the board. The CC signals must not cross plane splits."
- note added: "https://microchip.my.site.com/s/article/USB-Type-C-Layout-Recommendations"
- moved on the sheet: R2
